Commit message: update

File: resources/robots/limx_tron1/WF_TRON1A/urdf/robot.urdf (robot description, URDF)
Before this commit: robot point_foot, 10 links, 9 joints
Links:
- removed link limx_imu
Joints:
- removed joint limx_imu_joint
- joint abad_L_Joint: limit lower=-0.38397 upper=1.39626 effort=80.0 velocity=20.0 -> lower=-0.38397 upper=1.39626 effort=80.0 velocity=18.0
- joint abad_R_Joint: limit lower=-1.39626 upper=0.38397 effort=80.0 velocity=20.0 -> lower=-1.39626 upper=0.38397 effort=80.0 velocity=18.0
- joint hip_L_Joint: limit lower=-1.012291 upper=1.396263 effort=80.0 velocity=20.0 -> lower=-1.012291 upper=1.396263 effort=80.0 velocity=18.0
- joint hip_R_Joint: limit lower=-1.396263 upper=1.012291 effort=80.0 velocity=20.0 -> lower=-1.396263 upper=1.012291 effort=80.0 velocity=18.0
- joint knee_L_Joint: limit lower=-0.872665 upper=1.361357 effort=80 velocity=20 -> lower=-0.872665 upper=1.361357 effort=80 velocity=18
- joint knee_R_Joint: limit lower=-1.361357 upper=0.872665 effort=80 velocity=20 -> lower=-1.361357 upper=0.872665 effort=80 velocity=18
- joint wheel_L_Joint: limit lower=-100000 upper=100000 effort=40 velocity=40 -> lower=-100000 upper=100000 effort=40 velocity=18
- joint wheel_R_Joint: limit lower=-100000 upper=100000 effort=40 velocity=40 -> lower=-100000 upper=100000 effort=40 velocity=18
